Commit message: Controller

File: urdf/AllPart_ROS_1.xacro (robot description, xacro)
@@ -6,32 +6,4 @@
   name="AllPart_ROS_Z-up_W">
   <link
-    name="base_link">
-    <inertial>
-      <origin xyz="0 0 0" rpy="0 0 0" />
-      <mass value="0.01" />
-      <inertia ixx="0.01" ixy="0" ixz="0" iyy="0.01" iyz="0" izz="0.01" />
-    </inertial>
-    <visual>
-      <origin xyz="0 0 0" rpy="0 0 0" />
-      <geometry>
-        <box size="0.01 0.01 0.01" />
-      </geometry>
-      <material name="gray">
-        <color rgba="0.5 0.5 0.5 1" />
-      </material>
-    </visual>
-    <collision>
-      <origin xyz="0 0 0" rpy="0 0 0" />
-      <geometry>
-        <box size="0.01 0.01 0.01" />
-      </geometry>
-    </collision>
-  </link>
-  <joint name="base_joint" type="fixed">
-    <parent link="base_link" />
-    <child link="Origin_link" />
-    <origin xyz="0 0 0" rpy="0 0 0" />
-  </joint>
-  <link
     name="Origin_link">
     <inertial>
@@ -55,5 +27,5 @@
       <geometry>
         <mesh
-          filename="meshes/Origin_link.STL" />
+          filename="file:///home/nine/ballzaros_ws/src/ballzaros/meshes/Origin_link.STL" />
       </geometry>
       <material
@@ -69,5 +41,5 @@
       <geometry>
         <mesh
-          filename="meshes/Origin_link.STL" />
+          filename="file:///home/nine/ballzaros_ws/src/ballzaros/meshes/Origin_link.STL" />
       </geometry>
     </collision>
@@ -95,5 +67,5 @@
       <geometry>
         <mesh
-          filename="meshes/Left_Wheel_Link.STL" />
+          filename="file:///home/nine/ballzaros_ws/src/ballzaros/meshes/Left_Wheel_Link.STL" />
       </geometry>
       <material
@@ -109,5 +81,5 @@
       <geometry>
         <mesh
-          filename="meshes/Left_Wheel_Link.STL" />
+          filename="file:///home/nine/ballzaros_ws/src/ballzaros/meshes/Left_Wheel_Link.STL" />
       </geometry>
     </collision>
@@ -148,5 +120,5 @@
       <geometry>
         <mesh
-          filename="meshes/Right_Wheel_Link.STL" />
+          filename="file:///home/nine/ballzaros_ws/src/ballzaros/meshes/Right_Wheel_Link.STL" />
       </geometry>
       <material
@@ -162,5 +134,5 @@
       <geometry>
         <mesh
-          filename="meshes/Right_Wheel_Link.STL" />
+          filename="file:///home/nine/ballzaros_ws/src/ballzaros/meshes/Right_Wheel_Link.STL" />
       </geometry>
     </collision>
@@ -201,5 +173,5 @@
       <geometry>
         <mesh
-          filename="meshes/Lidar_Front_Link.STL" />
+          filename="file:///home/nine/ballzaros_ws/src/ballzaros/meshes/Lidar_Front_Link.STL" />
       </geometry>
       <material
@@ -215,5 +187,5 @@
       <geometry>
         <mesh
-          filename="meshes/Lidar_Front_Link.STL" />
+          filename="file:///home/nine/ballzaros_ws/src/ballzaros/meshes/Lidar_Front_Link.STL" />
       </geometry>
     </collision>
@@ -254,5 +226,5 @@
       <geometry>
         <mesh
-          filename="meshes/Lidar_Back_Link.STL" />
+          filename="file:///home/nine/ballzaros_ws/src/ballzaros/meshes/Lidar_Back_Link.STL" />
       </geometry>
       <material
@@ -268,5 +240,5 @@
       <geometry>
         <mesh
-          filename="meshes/Lidar_Back_Link.STL" />
+          filename="file:///home/nine/ballzaros_ws/src/ballzaros/meshes/Lidar_Back_Link.STL" />
       </geometry>
     </collision>
@@ -307,5 +279,5 @@
       <geometry>
         <mesh
-          filename="meshes/Cam_Front_Link.STL" />
+          filename="file:///home/nine/ballzaros_ws/src/ballzaros/meshes/Cam_Front_Link.STL" />
       </geometry>
       <material
@@ -321,5 +293,5 @@
       <geometry>
         <mesh
-          filename="meshes/Cam_Front_Link.STL" />
+          filename="file:///home/nine/ballzaros_ws/src/ballzaros/meshes/Cam_Front_Link.STL" />
       </geometry>
     </collision>
@@ -360,5 +332,5 @@
       <geometry>
         <mesh
-          filename="meshes/Cam_Back_Link.STL" />
+          filename="file:///home/nine/ballzaros_ws/src/ballzaros/meshes/Cam_Back_Link.STL" />
       </geometry>
       <material
@@ -374,5 +346,5 @@
       <geometry>
         <mesh
-          filename="meshes/Cam_Back_Link.STL" />
+          filename="file:///home/nine/ballzaros_ws/src/ballzaros/meshes/Cam_Back_Link.STL" />
       </geometry>
     </collision>
@@ -413,5 +385,5 @@
       <geometry>
         <mesh
-          filename="meshes/IMU_Link.STL" />
+          filename="file:///home/nine/ballzaros_ws/src/ballzaros/meshes/IMU_Link.STL" />
       </geometry>
       <material
@@ -427,5 +399,5 @@
       <geometry>
         <mesh
-          filename="meshes/IMU_Link.STL" />
+          filename="file:///home/nine/ballzaros_ws/src/ballzaros/meshes/IMU_Link.STL" />
       </geometry>
     </collision>
@@ -506,3 +478,23 @@
     </sensor>
   </gazebo>
+  <gazebo>
+    <plugin name='diff_drive' filename='libgazebo_ros_diff_drive.so'>
+      <!-- wheels -->
+      <left_joint>Left_Motor</left_joint>
+      <right_joint>Right_Motor</right_joint>
+      <!-- kinematics -->
+      <wheel_separation>0.26</wheel_separation>
+      <wheel_diameter>0.2</wheel_diameter>
+      <!-- limits -->
+  <max_wheel_torque>5000</max_wheel_torque>
+  <max_wheel_acceleration>2.0</max_wheel_acceleration>
+      <!-- output -->
+      <publish_odom>true</publish_odom>
+      <publish_odom_tf>true</publish_odom_tf>
+      <publish_wheel_tf>false</publish_wheel_tf>
+  <odometry_frame>odom</odometry_frame>
+  <robot_base_frame>base_link</robot_base_frame>
+  <cmd_vel_topic>cmd_vel</cmd_vel_topic>
+    </plugin>
+  </gazebo>
 </robot>
