Commit message: 30/9/2546

File: urdf/AllPart_ROS_1.xacro (robot description, xacro)
@@ -9,8 +9,8 @@
     <inertial>
       <origin
-        xyz="-0.0026663 -0.014052 0.44571"
-        rpy="0 0 0" />
-      <mass
-        value="75.301" />
+        xyz="0 0 -50"
+        rpy="0 0 0" />
+      <mass
+        value="5" />
       <inertia
         ixx="2.5951"
@@ -96,5 +96,5 @@
       link="Left_Wheel_Link" />
     <axis
-      xyz="0 0 -1" />
+      xyz="0 0 1" />
   </joint>
   <link
@@ -487,6 +487,6 @@
       <wheel_diameter>0.1</wheel_diameter>
       <!-- limits -->
-  <max_wheel_torque>5000</max_wheel_torque>
-  <max_wheel_acceleration>1000.0</max_wheel_acceleration>
+  <max_wheel_torque>0.5</max_wheel_torque>
+  <max_wheel_acceleration>1.0</max_wheel_acceleration>
       <!-- output -->
       <publish_odom>true</publish_odom>
@@ -498,3 +498,17 @@
     </plugin>
   </gazebo>
+    <!-- กำหนด physics ให้ล้อซ้าย -->
+  <gazebo reference="Left_Wheel_Link">
+    <mu1>3.0</mu1>
+    <mu2>3.0</mu2>
+    <kp>100000.0</kp>
+    <kd>1.0</kd>
+  </gazebo>
+  <!-- กำหนด physics ให้ล้อขวา -->
+  <gazebo reference="Right_Wheel_Link">
+    <mu1>3.0</mu1>
+    <mu2>3.0</mu2>
+    <kp>100000.0</kp>
+    <kd>1.0</kd>
+  </gazebo>
 </robot>
